File: optoprototype.sch (KiCad schematic (older format))
At the start: 36 parts, among them U1 LM393, U2 EL357N-D, U3 EL357N-D

Commit message: opto isolator prototype
Parts:
- removed GND_in1: GND_in, symbol Connector:Conn_01x01_Male
- removed GND_out1: GND_out, symbol Connector:Conn_01x01_Male
- removed In1: In1, symbol Connector:Conn_01x01_Male
- removed Out1: Out1, symbol Connector:Conn_01x01_Male
- removed Out2: Out2, symbol Connector:Conn_01x01_Male
- removed TX_485: TX_485, symbol Connector:Conn_01x01_Male
- removed V+_in1: V+_in, symbol Connector:Conn_01x01_Male
- removed V+_out1: V+_out, symbol Connector:Conn_01x01_Male
- removed VPU_out1: VPU_out, symbol Connector:Conn_01x01_Male
- added Input1: Input, Connector_PinHeader_2.54mm:PinHeader_1x04_P2.54mm_Vertical, symbol Connector:Conn_01x04_Female
- added Output1: Output, Connector_PinHeader_2.54mm:PinHeader_1x05_P2.54mm_Vertical, symbol Connector:Conn_01x05_Female
- C1, C10, C2, C3, C4, C5, C6, C7, C8, C9: footprint (none) -> Capacitor_SMD:C_0805_2012Metric_Pad1.18x1.45mm_HandSolder
- D1, D2: footprint Diode_THT:D_DO-35_SOD27_P7.62mm_Horizontal -> Diode_SMD:D_SOD-323
- R1, R10, R12, R2, R3, R4, R6, R7, R8, R9: footprint (none) -> Resistor_SMD:R_0805_2012Metric_Pad1.20x1.40mm_HandSolder
- R11, R5: footprint (none) -> Potentiometer_SMD:Potentiometer_Bourns_3214W_Vertical
- U1: footprint (none) -> Package_SO:SOP-8_5.28x5.23mm_P1.27mm
- U2, U3: footprint Package_DIP:DIP-4_W7.62mm -> Package_SO:SO-4_4.4x3.9mm_P2.54mm
Connections:
- net GND_in: now also Input1.4 (Pin_4)
- net GND_out: now also Output1.5 (Pin_5)
- net In1: now also Input1.2 (Pin_2)
- net In2: now also R7.1, Input1.3 (Pin_3); no longer R6.2, U1.1
- net Out1: now also R6.2, U1.1, Output1.3 (Pin_3); no longer R7.1
- net Out2: now also Output1.4 (Pin_4)
- net V+_in: now also Input1.1 (Pin_1)
- net V+_out: now also Output1.1 (Pin_1)
- net VPU_out: now also Output1.2 (Pin_2)
